Commit message: Imported upstream version '0.0.2' of 'upstream'

File: carl_description/robots/carl.urdf (robot description, URDF)
Before this commit: robot carl, 47 links, 46 joints
Links:
- added link camera_depth_frame, mass 0.01
- added link camera_depth_optical_frame, mass 0.001
- added link camera_rgb_frame, mass 0.001
- added link camera_rgb_optical_frame, mass 0.001
- link camera_link: geometry collision box size=0.0730 .2760 0.0720; visual mesh filename=package://carl_description/meshes/asus_xtion_pro_live.min.d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 scale=0.001 0.001 0.001
Joints:
- added joint camera_depth_joint: type fixed, parent camera_link, child camera_depth_frame, origin xyz=0 0.049 0 rpy=0 0 0
- added joint camera_depth_optical_joint: type fixed, parent camera_depth_frame, child camera_depth_optical_frame, origin xyz=0 0 0 rpy=-1.57079632679 0 -1.57079632679
- added joint camera_rgb_joint: type fixed, parent camera_link, child camera_rgb_frame, origin xyz=0 0.022 0 rpy=0 0 0
- added joint camera_rgb_optical_joint: type fixed, parent camera_rgb_frame, child camera_rgb_optical_frame, origin xyz=0 0 0 rpy=-1.57079632679 0 -1.57079632679
- joint camera_joint: origin xyz=-0.016 -0.008 0.018 rpy=0 -1.5708 0 -> xyz=-0.016 -0.008 0.018 rpy=0 -1.53 0

File: carl_description/urdf/carl_base/carl_asus_camera_mount.urdf.xacro (robot description, xacro)
@@ -71,5 +71,6 @@
     </link>
     <xacro:sensor_asus_xtion_pro parent="asus_mount_link">
-      <origin xyz="-0.016 -0.008 0.018" rpy="0 -1.5708 0" />
+      <!-- <origin xyz="-0.016 -0.008 0.018" rpy="0 -1.5708 0" /> -->
+      <origin xyz="-0.016 -0.008 0.018" rpy="0 -1.53 0" />
     </xacro:sensor_asus_xtion_pro>
     <joint name="right_rear_strut_asus_lift_joint" type="fixed">

File: carl_description/urdf/sensors/asus_xtion_pro.urdf.xacro (robot description, xacro)
@@ -12,23 +12,71 @@
       <child link="camera_link" />
     </joint>
-    <link name="camera_link">
-      <visual>
-        <origin xyz="-0.01 0 0" rpy="${-M_PI/2} -${M_PI} ${-M_PI/2}" />
-        <geometry>
-          <mesh filename="package://carl_description/meshes/asus_xtion_pro_live.min.dae" scale="${M_SCALE} ${M_SCALE} ${M_SCALE}" />
-        </geometry>
-      </visual>
-      <collision>
-        <origin xyz="0.0 0.0 0.0" rpy="0 0 0" />
-        <geometry>
-        <box size="0.0830 .2760 0.0720" />
+  <link name="camera_link">
+    <inertial>
+      <mass value="0.01" />
+      <origin xyz="0 0 0" />
+      <inertia ixx="0.001" ixy="0.0" ixz="0.0" iyy="0.001" iyz="0.0" izz="0.001" />
+    </inertial>
+    <visual>
+      <origin xyz=" 0 0 0 " rpy="${-M_PI/2} -${M_PI} ${-M_PI/2}" />
+      <geometry>
+        <mesh filename="package://carl_description/meshes/asus_xtion_pro_live.min.dae" scale="${M_SCALE} ${M_SCALE} ${M_SCALE}" />
       </geometry>
-      </collision>
-      <inertial>
-        <mass value="0.01" />
-        <origin xyz="0 0 0" />
-        <inertia ixx="0.001" ixy="0.0" ixz="0.0" iyy="0.001" iyz="0.0" izz="0.001" />
-      </inertial>
-    </link>
+    </visual>
+    <collision>
+      <origin xyz="0.0 0.0 0.0" rpy="0 0 0" />
+      <geometry>
+        <box size="0.0730 .2760 0.0720"/>
+      </geometry>
+    </collision>
+  </link>
+  <joint name="camera_depth_joint" type="fixed">
+    <origin xyz="0 0.049 0" rpy="0 0 0" />
+    <parent link="camera_link" />
+    <child link="camera_depth_frame" />
+  </joint>
+  <link name="camera_depth_frame">
+    <inertial>
+      <mass value="0.01" />
+      <origin xyz="0 0 0" />
+      <inertia ixx="0.001" ixy="0.0" ixz="0.0" iyy="0.001" iyz="0.0" izz="0.001" />
+    </inertial>
+  </link>
+  <joint name="camera_depth_optical_joint" type="fixed">
+    <origin xyz="0 0 0" rpy="${-M_PI/2} 0 ${-M_PI/2}" />
+    <parent link="camera_depth_frame" />
+    <child link="camera_depth_optical_frame" />
+  </joint>
+  <link name="camera_depth_optical_frame">
+    <inertial>
+      <mass value="0.001" />
+      <origin xyz="0 0 0" />
+      <inertia ixx="0.0001" ixy="0.0" ixz="0.0" iyy="0.0001" iyz="0.0" izz="0.0001" />
+    </inertial>
+  </link>
+  <joint name="camera_rgb_joint" type="fixed">
+    <origin xyz="0 0.022 0" rpy="0 0 0" />
+    <parent link="camera_link" />
+    <child link="camera_rgb_frame" />
+  </joint>
+  <link name="camera_rgb_frame">
+    <inertial>
+      <mass value="0.001" />
+      <origin xyz="0 0 0" />
+      <inertia ixx="0.0001" ixy="0.0" ixz="0.0" iyy="0.0001" iyz="0.0" izz="0.0001" />
+    </inertial>
+  </link>
+  <joint name="camera_rgb_optical_joint" type="fixed">
+    <origin xyz="0 0 0" rpy="${-M_PI/2} 0 ${-M_PI/2}" />
+    <parent link="camera_rgb_frame" />
+    <child link="camera_rgb_optical_frame" />
+  </joint>
+  <link name="camera_rgb_optical_frame">
+    <inertial>
+      <mass value="0.001" />
+      <origin xyz="0 0 0" />
+      <inertia ixx="0.0001" ixy="0.0" ixz="0.0" iyy="0.0001" iyz="0.0" izz="0.0001" />
+    </inertial>
+  </link>
   </xacro:macro>
 </robot>

Commit message: Imported upstream version '0.0.6' of 'upstream'

File: carl_description/robots/carl.urdf (robot description, URDF)
Before this commit: robot carl, 51 links, 50 joints
Links:
- link back_cover_link: geometry collision box size=.05 .45 1.56; visual mesh filename=package://carl_description/meshes/back_cover.min.dae scale=0.0254 0.0254 0.0254

File: carl_description/urdf/carl_base/carl_covers.urdf.xacro (robot description, xacro)
@@ -43,8 +43,14 @@
       </visual>
       <collision>
+        <origin xyz=".025 0 .8" rpy="0 0 0" />
+        <geometry>
+          <box size=".05 .45 1.56" />
+        </geometry>
+        <!--
         <origin xyz="0 0 0" rpy="0 0 0" />
         <geometry>
           <mesh scale="${M_SCALE} ${M_SCALE} ${M_SCALE}" filename="package://carl_description/meshes/back_cover.stl" />
         </geometry>
+        -->
       </collision>
     </link>
